File: Board/RailcomSwitchChanger.kicad_pcb (KiCad board)
At the start: 2 copper layers, 72 x 68 mm, 85 parts, among them J1 RAIL_IN, J11 UPDI, J12 Serial, J13 PROG, J14 SW_OUT, J15 Debug, J16 LOCK_INPUT, J17 LOCK_INPUT_TOMIX, J2 RAIL_OUT, Q1 SSM3K7002BFU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

Commit message: Board Rev.2
Parts:
- added R42: 104, footprint:R_1608, F.Cu at (167.5, 76.2)
Routing:
- net GND: track 477.0 -> 479.3 mm
- net Net-(Q15-Pad1): track 2.11 -> 4.12 mm
- net Net-(Q13-Pad1): track 28.7 -> 27.0 mm
Other:
- board text added: "Rev.2 2022.08"
- board text removed: "Rev.1 2022.05"
