File: Board/rsc_mcu.sch (KiCad schematic (older format))
At the start: 51 parts, among them J11 UPDI, J12 Serial, J13 PROG, J14 SW_OUT, J15 Debug, J16 LOCK_INPUT, J17 LOCK_INPUT_TOMIX, Q11 FDS4897C, Q12 FDS4897C, Q13 2SC4116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

Commit message: Board Rev.2
Parts:
- added R42: 104, footprint:R_1608, symbol Device:R
Connections:
- net GND: now also R42.2
- net at Q15.1 (B), R41.1: now also R42.1
Changed lines of the file:
@@
 L power:GND #PWR0139
 U 1 1 61BC4FB1
-P 15100 9400
-F 0 "#PWR0139" H 15100 9150 50  0001 C CNN
-F 1 "GND" H 15105 9227 50  0000 C CNN
-F 2 "" H 15100 9400 50  0001 C CNN
-F 3 "" H 15100 9400 50  0001 C CNN
-	1    15100 9400
+P 15100 9600
+F 0 "#PWR0139" H 15100 9350 50  0001 C CNN
+F 1 "GND" H 15105 9427 50  0000 C CNN
+F 2 "" H 15100 9600 50  0001 C CNN
+F 3 "" H 15100 9600 50  0001 C CNN
+	1    15100 9600
 	1    0    0    -1
 $EndComp
-Wire Wire Line
-	15100 9400 15100 9200
 Wire Wire Line
 	15100 8800 15100 8600
@@
 $EndComp
 Wire Wire Line
-	14600 9000 14800 9000
+	14600 9000 14700 9000
 $Comp
 L Connector_Generic:Conn_01x03 J16
@@
 	13050 9100 13300 9100
 Wire Wire Line
-	13300 9100 13300 9400
-Wire Wire Line
 	13050 8900 13300 8900
 Wire Wire Line
@@
 L power:GND #PWR0140
 U 1 1 61C2DFA1
-P 13300 9400
-F 0 "#PWR0140" H 13300 9150 50  0001 C CNN
-F 1 "GND" H 13305 9227 50  0000 C CNN
-F 2 "" H 13300 9400 50  0001 C CNN
-F 3 "" H 13300 9400 50  0001 C CNN
-	1    13300 9400
+P 13300 9600
+F 0 "#PWR0140" H 13300 9350 50  0001 C CNN
+F 1 "GND" H 13305 9427 50  0000 C CNN
+F 2 "" H 13300 9600 50  0001 C CNN
+F 3 "" H 13300 9600 50  0001 C CNN
+	1    13300 9600
 	1    0    0    -1
 $EndComp
@@
 	1    0    0    -1
 $EndComp
+$Comp
+L Device:R R42
+U 1 1 62F510BE
+P 14700 9300
+F 0 "R42" H 14770 9346 50  0000 L CNN
+F 1 "104" H 14770 9255 50  0000 L CNN
+F 2 "footprint:R_1608" V 14630 9300 50  0001 C CNN
+F 3 "~" H 14700 9300 50  0001 C CNN
+	1    14700 9300
+	1    0    0    -1
+$EndComp
+$Comp
+L power:GND #PWR?
+U 1 1 62F627C8
+P 14700 9600
+F 0 "#PWR?" H 14700 9350 50  0001 C CNN
+F 1 "GND" H 14705 9427 50  0000 C CNN
+F 2 "" H 14700 9600 50  0001 C CNN
+F 3 "" H 14700 9600 50  0001 C CNN
+	1    14700 9600
+	1    0    0    -1
+$EndComp
+Wire Wire Line
+	14700 9600 14700 9450
+Wire Wire Line
+	14700 9150 14700 9000
+Connection ~ 14700 9000
+Wire Wire Line
+	14700 9000 14800 9000
+Wire Wire Line
+	15100 9200 15100 9600
+Wire Wire Line
+	13300 9100 13300 9600
 $EndSCHEMATC
